Commit message: Initial commit: dual arm ROS2 workspace

File: src/onrobot_description/urdf/onrobot_macro.xacro (robot description, xacro)
@@ -28,5 +28,5 @@
         </xacro:if>
         <!-- Define the OnRobot gripper hardware interface for ROS 2 control -->
-        <ros2_control name="OnRobotGripper" type="actuator">
+        <ros2_control name="${prefix}OnRobotGripper" type="actuator">
             <hardware>
                 <xacro:if value="${sim_gazebo}">

File: src/ur_onrobot/ur_onrobot_description/urdf/ur_onrobot.urdf.xacro (robot description, xacro)
@@ -1,50 +1,37 @@
 <?xml version="1.0"?>
-<robot xmlns:xacro="http://ros.org/wiki/xacro">
-  <xacro:include filename="$(find ur_description)/urdf/ur_macro.xacro"/>
-  <xacro:include filename="$(find onrobot_description)/urdf/onrobot_rg2_macro.xacro"/>
-  <xacro:macro name="ur_onrobot" params="
-    parent
-    robot_ip
-    ur_type
-    onrobot_type
-    tf_prefix
-    use_fake_hardware
-    joint_limits_parameters_file
-    kinematics_parameters_file
-    physical_parameters_file
-    visual_parameters_file
-    script_filename
-    output_recipe_filename
-    input_recipe_filename
-    origin_xyz:='0 0 0'
-    origin_rpy:='0 0 0'"
-  >
-    <joint name="${tf_prefix}base_joint" type="fixed">
-      <parent link="${parent}" />
-      <child link="${tf_prefix}base_link" />
-      <origin xyz="${origin_xyz}" rpy="${origin_rpy}" />
-    </joint>
-    <xacro:ur_robot
-      name="${tf_prefix}ur"
-      tf_prefix="${tf_prefix}"
-      parent="${parent}"
-      joint_limits_parameters_file="${joint_limits_parameters_file}"
-      kinematics_parameters_file="${kinematics_parameters_file}"
-      physical_parameters_file="${physical_parameters_file}"
-      visual_parameters_file="${visual_parameters_file}"
-      use_fake_hardware="${use_fake_hardware}"
-      robot_ip="${robot_ip}"
-      script_filename="${script_filename}"
-      output_recipe_filename="${output_recipe_filename}"
-      input_recipe_filename="${input_recipe_filename}"
-    >
-      <origin xyz="0 0 0" rpy="0 0 0" />
-    </xacro:ur_robot>
-    <joint name="${tf_prefix}ur_to_onrobot" type="fixed">
-      <parent link="${tf_prefix}tool0" />
-      <child link="${tf_prefix}onrobot_base_link" />
-      <origin xyz="0 0 0" rpy="0 0 0" />
-    </joint>
-    <xacro:onrobot_rg2 prefix="${tf_prefix}"/>
-  </xacro:macro>
+<robot name="ur_onrobot" xmlns:xacro="http://ros.org/wiki/xacro">
+    <!-- Arguments -->
+    <xacro:arg name="robot_ip" default="192.168.56.101"/>
+    <xacro:arg name="ur_type" default="ur3e"/>
+    <xacro:arg name="onrobot_type" default="rg2"/>
+    <xacro:arg name="tf_prefix" default=""/>
+    <xacro:arg name="name" default="ur_onrobot"/>
+    <xacro:arg name="use_fake_hardware" default="false"/>
+    <xacro:arg name="joint_limits_parameters_file" default="$(find ur_description)/config/$(arg ur_type)/joint_limits.yaml"/>
+    <xacro:arg name="kinematics_parameters_file" default="$(find ur_description)/config/$(arg ur_type)/default_kinematics.yaml"/>
+    <xacro:arg name="physical_parameters_file" default="$(find ur_description)/config/$(arg ur_type)/physical_parameters.yaml"/>
+    <xacro:arg name="visual_parameters_file" default="$(find ur_description)/config/$(arg ur_type)/visual_parameters.yaml"/>
+    <xacro:arg name="script_filename" default="$(find ur_client_library)/resources/external_control.urscript"/>
+    <xacro:arg name="input_recipe_filename" default="$(find ur_robot_driver)/resources/rtde_input_recipe.txt"/>
+    <xacro:arg name="output_recipe_filename" default="$(find ur_robot_driver)/resources/rtde_output_recipe.txt"/>
+    <xacro:include filename="$(find ur_onrobot_description)/urdf/ur_onrobot_macro.xacro"/>
+    <link name="world"/>
+    <!--This will create the scene where the robot is located in-->
+    <xacro:ur_onrobot
+        parent="world"
+        robot_ip="$(arg robot_ip)"
+        ur_type="$(arg ur_type)"
+        onrobot_type="$(arg onrobot_type)"
+        tf_prefix="$(arg tf_prefix)"
+        use_fake_hardware="$(arg use_fake_hardware)"
+        joint_limits_parameters_file="$(arg joint_limits_parameters_file)"
+        kinematics_parameters_file="$(arg kinematics_parameters_file)"
+        physical_parameters_file="$(arg physical_parameters_file)"
+        visual_parameters_file="$(arg visual_parameters_file)"
+        script_filename="$(arg script_filename)"
+        output_recipe_filename="$(arg output_recipe_filename)"
+        input_recipe_filename="$(arg input_recipe_filename)"
+        >
+        <origin xyz="0 0 1" rpy="0 0 0" />
+    </xacro:ur_onrobot>
 </robot>

File: src/ur_onrobot/ur_onrobot_description/urdf/ur_onrobot_macro.xacro (robot description, xacro)
@@ -19,8 +19,9 @@
         output_recipe_filename
         input_recipe_filename
+        include_ros2_control:=false
         ">
         <xacro:ur_robot
             robot_ip="${robot_ip}"
-            name="${ur_type}"
+            name="${tf_prefix}${ur_type}"
             parent="${parent}"
             tf_prefix="${tf_prefix}"

File: src/ur_onrobot/ur_onrobot_moveit_config/srdf/dual_ur_onrobot.srdf.xacro (robot description, xacro)
@@ -1,42 +1,71 @@
 <?xml version="1.0" encoding="UTF-8"?>
 <robot name="dual_ur_onrobot" xmlns:xacro="http://ros.org/wiki/xacro">
-    <xacro:include filename="$(find ur_onrobot_moveit_config)/config/ur_onrobot.srdf.xacro" />
+    <!-- Include file macro SRDF -->
+    <xacro:include filename="$(find ur_onrobot_moveit_config)/srdf/ur_onrobot_macro.srdf.xacro" />
+    <!-- Gọi macro cho tay trái và tay phải -->
     <xacro:ur_onrobot_srdf name="ur_onrobot" prefix="left_" />
     <xacro:ur_onrobot_srdf name="ur_onrobot" prefix="right_" />
-    <group_state name="left_home" group="left_ur_onrobot_manipulator">
-        <joint name="left_elbow_joint" value="0" />
-        <joint name="left_shoulder_lift_joint" value="-1.5707" />
-        <joint name="left_shoulder_pan_joint" value="0" />
-        <joint name="left_wrist_1_joint" value="0" />
-        <joint name="left_wrist_2_joint" value="0" />
+    <!-- Tư thế tự định nghĩa cho TAY TRÁI -->
+    <group_state name="left_scan_camera" group="left_ur_onrobot_manipulator">
+        <joint name="left_elbow_joint" value="1.5" />
+        <joint name="left_shoulder_lift_joint" value="-2.0" />
+        <joint name="left_shoulder_pan_joint" value="1.0" />
+        <joint name="left_wrist_1_joint" value="-1.0" />
+        <joint name="left_wrist_2_joint" value="1.57" />
         <joint name="left_wrist_3_joint" value="0" />
     </group_state>
-    <group_state name="left_up" group="left_ur_onrobot_manipulator">
-        <joint name="left_elbow_joint" value="0" />
-        <joint name="left_shoulder_lift_joint" value="-1.5707" />
-        <joint name="left_shoulder_pan_joint" value="0" />
-        <joint name="left_wrist_1_joint" value="-1.5707" />
-        <joint name="left_wrist_2_joint" value="0" />
-        <joint name="left_wrist_3_joint" value="0" />
+    <group_state name="gap_vat" group="left_ur_onrobot_manipulator">
+        <joint name="left_shoulder_pan_joint" value="1.4312"/>
+        <joint name="left_shoulder_lift_joint" value="-0.3665"/>
+        <joint name="left_elbow_joint" value="0.0524"/>
+        <joint name="left_wrist_1_joint" value="-1.1519"/>
+        <joint name="left_wrist_2_joint" value="-1.7802"/>
+        <joint name="left_wrist_3_joint" value="0.0000"/>
     </group_state>
-    <group_state name="right_home" group="right_ur_onrobot_manipulator">
-        <joint name="right_elbow_joint" value="0" />
-        <joint name="right_shoulder_lift_joint" value="-1.5707" />
-        <joint name="right_shoulder_pan_joint" value="0" />
-        <joint name="right_wrist_1_joint" value="0" />
-        <joint name="right_wrist_2_joint" value="0" />
-        <joint name="right_wrist_3_joint" value="0" />
+    <group_state name="tha_vat" group="left_ur_onrobot_manipulator">
+        <joint name="left_shoulder_pan_joint" value="-1.8500"/>
+        <joint name="left_shoulder_lift_joint" value="-0.3665"/>
+        <joint name="left_elbow_joint" value="0.0175"/>
+        <joint name="left_wrist_1_joint" value="-1.1170"/>
+        <joint name="left_wrist_2_joint" value="-1.5708"/>
+        <joint name="left_wrist_3_joint" value="0.0000"/>
     </group_state>
-    <group_state name="right_up" group="right_ur_onrobot_manipulator">
-        <joint name="right_elbow_joint" value="0" />
-        <joint name="right_shoulder_lift_joint" value="-1.5707" />
-        <joint name="right_shoulder_pan_joint" value="0" />
-        <joint name="right_wrist_1_joint" value="-1.5707" />
-        <joint name="right_wrist_2_joint" value="0" />
-        <joint name="right_wrist_3_joint" value="0" />
+    <!-- Tư thế tự định nghĩa cho TAY PHẢI -->
+    <group_state name="gap_vat" group="right_ur_onrobot_manipulator">
+        <joint name="right_shoulder_pan_joint" value="-1.3265"/>
+        <joint name="right_shoulder_lift_joint" value="-2.2689"/>
+        <joint name="right_elbow_joint" value="-1.0821"/>
+        <joint name="right_wrist_1_joint" value="-1.2915"/>
+        <joint name="right_wrist_2_joint" value="1.6057"/>
+        <joint name="right_wrist_3_joint" value="0.0000"/>
     </group_state>
+    <group_state name="tha_vat" group="right_ur_onrobot_manipulator">
+        <joint name="right_shoulder_pan_joint" value="3.2289"/>
+        <joint name="right_shoulder_lift_joint" value="-0.2269"/>
+        <joint name="right_elbow_joint" value="-0.3142"/>
+        <joint name="right_wrist_1_joint" value="-1.0297"/>
+        <joint name="right_wrist_2_joint" value="-1.5708"/>
+        <joint name="right_wrist_3_joint" value="0.0000"/>
+    </group_state>
+    <!-- Vô hiệu hóa va chạm giữa 2 đế robot -->
     <disable_collisions link1="left_base_link" link2="right_base_link" reason="FixedBase" />
     <disable_collisions link1="left_base_link_inertia" link2="right_base_link_inertia" reason="FixedBase" />
     <disable_collisions link1="left_base_link" link2="right_base_link_inertia" reason="FixedBase" />
     <disable_collisions link1="left_base_link_inertia" link2="right_base_link" reason="FixedBase" />
+    <!-- Vô hiệu hóa tự va chạm tay kẹp TAY TRÁI (left_) -->
+    <disable_collisions link1="left_right_inner_knuckle" link2="left_right_inner_finger" reason="Adjacent"/>
+    <disable_collisions link1="left_right_inner_finger" link2="left_right_outer_knuckle" reason="Never"/>
+    <disable_collisions link1="left_left_inner_knuckle" link2="left_left_inner_finger" reason="Adjacent"/>
+    <disable_collisions link1="left_left_inner_finger" link2="left_left_outer_knuckle" reason="Never"/>
+    <disable_collisions link1="left_left_inner_knuckle" link2="left_right_inner_knuckle" reason="Never"/>
+    <disable_collisions link1="left_left_inner_finger" link2="left_right_inner_finger" reason="Never"/>
+    <disable_collisions link1="left_left_outer_knuckle" link2="left_right_outer_knuckle" reason="Never"/>
+    <!-- Vô hiệu hóa tự va chạm tay kẹp TAY PHẢI (right_) -->
+    <disable_collisions link1="right_right_inner_knuckle" link2="right_right_inner_finger" reason="Adjacent"/>
+    <disable_collisions link1="right_right_inner_finger" link2="right_right_outer_knuckle" reason="Never"/>
+    <disable_collisions link1="right_left_inner_knuckle" link2="right_left_inner_finger" reason="Adjacent"/>
+    <disable_collisions link1="right_left_inner_finger" link2="right_left_outer_knuckle" reason="Never"/>
+    <disable_collisions link1="right_left_inner_knuckle" link2="right_right_inner_knuckle" reason="Never"/>
+    <disable_collisions link1="right_left_inner_finger" link2="right_right_inner_finger" reason="Never"/>
+    <disable_collisions link1="right_left_outer_knuckle" link2="right_right_outer_knuckle" reason="Never"/>
 </robot>

File: src/ur_onrobot/ur_onrobot_moveit_config/srdf/ur_onrobot_macro.srdf.xacro (robot description, xacro)
@@ -1,14 +1,6 @@
 <?xml version="1.0" encoding="UTF-8"?>
 <robot xmlns:xacro="http://wiki.ros.org/xacro">
-<!--This does not replace URDF, and is not an extension of URDF.
-    This is a format for representing semantic information about the robot structure.
-    A URDF file must exist for this robot as well, where the joints and the links that are referenced are defined
--->
   <xacro:macro name="ur_onrobot_srdf" params="name prefix">
-    <!--GROUPS - Representation of a set of joints and links. This can be useful for specifying DOF to plan for, defining arms, end effectors, etc-->
-    <!--LINKS - When a link is specified, the parent joint of that link (if it exists) is automatically included-->
-    <!--JOINTS - When a joint is specified, the child link of that joint (which will always exist) is automatically included-->
-    <!--CHAINS - When a chain is specified, all the links along the chain (including endpoints) are included in the group. Additionally, all the joints that are parents to included links are also included. This means that joints along the chain and the parent joint of the base link are included in the group-->
-    <!--SUBGROUPS - Groups can also be formed by referencing to already defined group names-->
+    <!-- GROUPS -->
     <group name="${prefix}${name}_gripper">
       <link name="${prefix}onrobot_base_link"/>
@@ -29,10 +21,10 @@
       <chain base_link="${prefix}base_link" tip_link="${prefix}gripper_tcp" />
     </group>
-    <!--GROUP STATES - Purpose - Define a named state for a particular group, in terms of joint values. This is useful to define states like 'folded arms'-->
+    <!-- GROUP STATES -->
     <group_state name="closed" group="${prefix}${name}_gripper">
-      <joint name="finger_width" value="0.0"/>
+      <joint name="${prefix}finger_width" value="0.0"/>
     </group_state>
     <group_state name="open" group="${prefix}${name}_gripper">
-      <joint name="finger_width" value="0.100"/>
+      <joint name="${prefix}finger_width" value="0.100"/>
     </group_state>
     <group_state name="${prefix}home" group="${prefix}${name}_manipulator">
@@ -60,8 +52,7 @@
       <joint name="${prefix}wrist_3_joint" value="-0.11" />
     </group_state>
-    <!--END EFFECTOR - Purpose - Represent information about an end effector.-->
+    <!-- END EFFECTOR -->
     <end_effector name="${prefix}${name}_gripper" parent_link="${prefix}gripper_tcp" group="${prefix}${name}_gripper" parent_group="${prefix}${name}_manipulator"/>
-    <!--VIRTUAL JOINT - Purpose - this element defines a virtual joint between a robot link and an external frame of reference (considered fixed with respect to the robot)-->
-    <!--DISABLE COLLISIONS - By default it is assumed that any link of the robot could potentially come into collision with any other link in the robot. This tag disables collision checking between a specified pair of links. -->
+    <!-- DISABLE COLLISIONS: Cánh tay UR -->
     <disable_collisions link1="${prefix}base_link" link2="${prefix}base_link_inertia" reason="Adjacent" />
     <disable_collisions link1="${prefix}base_link_inertia" link2="${prefix}shoulder_link" reason="Adjacent" />
@@ -75,4 +66,12 @@
     <disable_collisions link1="${prefix}wrist_1_link" link2="${prefix}wrist_3_link" reason="Never" />
     <disable_collisions link1="${prefix}wrist_2_link" link2="${prefix}wrist_3_link" reason="Adjacent" />
+    <!-- DISABLE COLLISIONS: Khớp nối tay kẹp OnRobot với Cánh tay UR -->
+    <disable_collisions link1="${prefix}tool0" link2="${prefix}onrobot_base_link" reason="Adjacent" />
+    <disable_collisions link1="${prefix}tool0" link2="${prefix}cable_connector_0" reason="Never" />
+    <disable_collisions link1="${prefix}tool0" link2="${prefix}cable_connector_1" reason="Never" />
+    <disable_collisions link1="${prefix}onrobot_base_link" link2="${prefix}wrist_1_link" reason="Never" />
+    <disable_collisions link1="${prefix}onrobot_base_link" link2="${prefix}wrist_2_link" reason="Never" />
+    <disable_collisions link1="${prefix}onrobot_base_link" link2="${prefix}wrist_3_link" reason="Adjacent" />
+    <!-- DISABLE COLLISIONS: Các bộ phận OnRobot Gripper -->
     <disable_collisions link1="${prefix}cable_connector_0" link2="${prefix}cable_connector_1" reason="Never"/>
     <disable_collisions link1="${prefix}cable_connector_0" link2="${prefix}left_inner_finger" reason="Never"/>
@@ -123,7 +122,4 @@
     <disable_collisions link1="${prefix}onrobot_base_link" link2="${prefix}right_inner_knuckle" reason="Adjacent"/>
     <disable_collisions link1="${prefix}onrobot_base_link" link2="${prefix}right_outer_knuckle" reason="Adjacent"/>
-    <disable_collisions link1="${prefix}onrobot_base_link" link2="${prefix}wrist_1_link" reason="Never"/>
-    <disable_collisions link1="${prefix}onrobot_base_link" link2="${prefix}wrist_2_link" reason="Never"/>
-    <disable_collisions link1="${prefix}onrobot_base_link" link2="${prefix}wrist_3_link" reason="Adjacent"/>
     <disable_collisions link1="${prefix}right_inner_finger" link2="${prefix}right_inner_knuckle" reason="Default"/>
     <disable_collisions link1="${prefix}right_inner_finger" link2="${prefix}right_outer_knuckle" reason="Adjacent"/>
