Commit message: Update src from 2tay_ws

File: src/ur_onrobot/ur_onrobot_description/urdf/dual_ur_onrobot.urdf.xacro (robot description, xacro)
@@ -30,5 +30,5 @@
         input_recipe_filename="$(arg input_recipe_filename)"
     >
-        <origin xyz="0.0 0.5 0.0" rpy="0.0 0.0 0.0" />
+        <origin xyz="0.0 0.25 0.0" rpy="0.0 0.0 0.0" />
     </xacro:ur_onrobot>
     <xacro:ur_onrobot
@@ -47,5 +47,5 @@
         input_recipe_filename="$(arg input_recipe_filename)"
     >
-        <origin xyz="0.0 -0.5 0.0" rpy="0.0 0.0 0.0" />
+        <origin xyz="0.0 -0.25 0.0" rpy="0.0 0.0 0.0" />
     </xacro:ur_onrobot>
 </robot>

File: src/ur_onrobot/ur_onrobot_moveit_config/srdf/dual_ur_onrobot.srdf.xacro (robot description, xacro)
@@ -6,4 +6,12 @@
     <xacro:ur_onrobot_srdf name="ur_onrobot" prefix="left_" />
     <xacro:ur_onrobot_srdf name="ur_onrobot" prefix="right_" />
+    <group name="dual_arms">
+    <group name="left_ur_onrobot_manipulator"/>
+    <group name="right_ur_onrobot_manipulator"/>
+    </group>
+    <group name="dual_grippers">
+    <group name="left_ur_onrobot_gripper"/>
+    <group name="right_ur_onrobot_gripper"/>
+    </group>
     <!-- Tư thế tự định nghĩa cho TAY TRÁI -->
     <group_state name="left_scan_camera" group="left_ur_onrobot_manipulator">

Commit message: Update 2tay_ws

File: src/ur_onrobot/ur_onrobot_description/urdf/dual_ur_onrobot.urdf.xacro (robot description, xacro)
@@ -30,5 +30,5 @@
         input_recipe_filename="$(arg input_recipe_filename)"
     >
-        <origin xyz="0.0 0.25 0.0" rpy="0.0 0.0 0.0" />
+        <origin xyz="0.0 0.3 0.0" rpy="0.0 0.0 0.0" />
     </xacro:ur_onrobot>
     <xacro:ur_onrobot
@@ -47,5 +47,5 @@
         input_recipe_filename="$(arg input_recipe_filename)"
     >
-        <origin xyz="0.0 -0.25 0.0" rpy="0.0 0.0 0.0" />
+        <origin xyz="0.0 -0.3 0.0" rpy="0.0 0.0 0.0" />
     </xacro:ur_onrobot>
 </robot>
