Commit message: Update src 2tay_ws

File: src/ur_onrobot/ur_onrobot_moveit_config/srdf/dual_ur_onrobot.srdf.xacro (robot description, xacro)
@@ -49,5 +49,5 @@
     </group_state>
     <group_state name="tha_vat" group="right_ur_onrobot_manipulator">
-        <joint name="right_shoulder_pan_joint" value="3.2289"/>
+        <joint name="right_shoulder_pan_joint" value="-1.8500"/>
         <joint name="right_shoulder_lift_joint" value="-0.2269"/>
         <joint name="right_elbow_joint" value="-0.3142"/>
